File: Davinci-Keyboard/Davinci-Keyboard.kicad_pcb (KiCad board)
At the start: 2 copper layers, 35 parts, among them J1 Conn_01x02, J2 USB_C_Receptacle_USB2.0_16P, Q1 MMBT3906, Q2 MMBT3906, Q3 MMBT3906, Q4 BSS138, Q5 BSS138, Q7 MMBT3906, SW1 BOOT, SW2 RST, U1 FDS4935A, U2 ESP32-S3-WROOM-1, U3 CH340K

Commit message: 20$越え
Parts:
- removed LDO1: ~, Package_TO_SOT_THT:TO-220-4_Horizontal_TabDown
- removed Q7: MMBT3906, Package_TO_SOT_SMD:SOT-23
- added C10: 0.01uF, Capacitor_SMD:C_0603_1608Metric_Pad1.08x0.95mm_HandSolder, B.Cu at (47.5, 82.6)
- added C11: 0.01uF, Capacitor_SMD:C_0603_1608Metric_Pad1.08x0.95mm_HandSolder, B.Cu at (80.1, 82.4)
- added C12: 0.01uF, Capacitor_SMD:C_0603_1608Metric_Pad1.08x0.95mm_HandSolder, B.Cu at (80.1, 89.3)
- added C13: 0.01uF, Capacitor_SMD:C_0603_1608Metric_Pad1.08x0.95mm_HandSolder, B.Cu at (61.7, 128.3)
- added C14: 0.01uF, Capacitor_SMD:C_0603_1608Metric_Pad1.08x0.95mm_HandSolder, B.Cu at (65.8, 128.3)
- added C9: 0.01uF, Capacitor_SMD:C_0603_1608Metric_Pad1.08x0.95mm_HandSolder, B.Cu at (47.5, 89.3)
- added D10: 1N4148W, Diode_SMD:D_SOD-123, B.Cu at (115.4, 41.7)
- added D11: 1N4148W, Diode_SMD:D_SOD-123, B.Cu at (158.3, 41.7)
- added D12: 1N4148W, Diode_SMD:D_SOD-123, B.Cu at (196.4, 41.7)
- added D13: 1N4148W, Diode_SMD:D_SOD-123, B.Cu at (239.2, 41.7)
- added D14: 1N4148W, Diode_SMD:D_SOD-123, B.Cu at (277.3, 41.7)
- added D15: 1N4148W, Diode_SMD:D_SOD-123, B.Cu at (320.2, 41.7)
- added D16: 1N4148W, Diode_SMD:D_SOD-123, B.Cu at (358.3, 41.7)
- added D17: 1N4148W, Diode_SMD:D_SOD-123, B.Cu at (115.4, 65.5)
- added D18: 1N4148W, Diode_SMD:D_SOD-123, B.Cu at (153.5, 65.5)
- added D19: 1N4148W, Diode_SMD:D_SOD-123, B.Cu at (191.6, 65.5)
- added D20: 1N4148W, Diode_SMD:D_SOD-123, B.Cu at (229.7, 65.5)
- added D21: 1N4148W, Diode_SMD:D_SOD-123, B.Cu at (267.8, 65.5)
- added D22: 1N4148W, Diode_SMD:D_SOD-123, B.Cu at (305.9, 65.5)
- added D23: 1N4148W, Diode_SMD:D_SOD-123, B.Cu at (344.0, 65.5)
- added D24: 1N4148W, Diode_SMD:D_SOD-123, B.Cu at (405.9, 41.7)
- added D25: 1N4148W, Diode_SMD:D_SOD-123, B.Cu at (134.4, 65.5)
- added D26: 1N4148W, Diode_SMD:D_SOD-123, B.Cu at (172.5, 65.5)
- added D27: 1N4148W, Diode_SMD:D_SOD-123, B.Cu at (210.6, 65.5)
- added D28: 1N4148W, Diode_SMD:D_SOD-123, B.Cu at (248.7, 65.5)
- added D29: 1N4148W, Diode_SMD:D_SOD-123, B.Cu at (286.8, 65.5)
- added D3: 1N4148W, Diode_SMD:D_SOD-123, B.Cu at (139.2, 41.7)
- added D30: 1N4148W, Diode_SMD:D_SOD-123, B.Cu at (324.9, 65.5)
- added D31: 1N4148W, Diode_SMD:D_SOD-123, B.Cu at (382.1, 65.5)
- added D32: 1N4148W, Diode_SMD:D_SOD-123, B.Cu at (120.2, 84.5)
- added D33: 1N4148W, Diode_SMD:D_SOD-123, B.Cu at (163.0, 84.5)
- added D34: 1N4148W, Diode_SMD:D_SOD-123, B.Cu at (201.1, 84.5)
- added D35: 1N4148W, Diode_SMD:D_SOD-123, B.Cu at (239.2, 84.5)
- added D36: 1N4148W, Diode_SMD:D_SOD-123, B.Cu at (277.3, 84.5)
- added D37: 1N4148W, Diode_SMD:D_SOD-123, B.Cu at (315.4, 84.5)
- added D38: 1N4148W, Diode_SMD:D_SOD-123, B.Cu at (334.5, 84.5)
- added D39: 1N4148W, Diode_SMD:D_SOD-123, B.Cu at (363.0, 65.5)
- added D4: 1N4148W, Diode_SMD:D_SOD-123, B.Cu at (177.3, 41.7)
- added D40: 1N4148W, Diode_SMD:D_SOD-123, B.Cu at (405.9, 65.5)
- added D41: 1N4148W, Diode_SMD:D_SOD-123, B.Cu at (144.0, 84.5)
- added D42: 1N4148W, Diode_SMD:D_SOD-123, B.Cu at (182.1, 84.5)
- added D43: 1N4148W, Diode_SMD:D_SOD-123, B.Cu at (220.2, 84.5)
- added D44: 1N4148W, Diode_SMD:D_SOD-123, B.Cu at (258.3, 84.5)
- added D45: 1N4148W, Diode_SMD:D_SOD-123, B.Cu at (296.4, 84.5)
- added D46: 1N4148W, Diode_SMD:D_SOD-123, B.Cu at (379.7, 94.0)
- added D47: 1N4148W, Diode_SMD:D_SOD-123, B.Cu at (122.5, 103.6)
- added D48: 1N4148W, Diode_SMD:D_SOD-123, B.Cu at (167.8, 103.6)
- added D49: 1N4148W, Diode_SMD:D_SOD-123, B.Cu at (205.9, 103.6)
- added D5: 1N4148W, Diode_SMD:D_SOD-123, B.Cu at (220.2, 41.7)
- added D50: 1N4148W, Diode_SMD:D_SOD-123, B.Cu at (244.0, 103.6)
- added D51: 1N4148W, Diode_SMD:D_SOD-123, B.Cu at (282.1, 103.6)
- added D52: 1N4148W, Diode_SMD:D_SOD-123, B.Cu at (320.2, 103.6)
- added D53: 1N4148W, Diode_SMD:D_SOD-123, B.Cu at (339.2, 103.6)
- added D54: 1N4148W, Diode_SMD:D_SOD-123, B.Cu at (353.5, 84.5)
- added D55: 1N4148W, Diode_SMD:D_SOD-123, B.Cu at (405.9, 84.5)
- added D56: 1N4148W, Diode_SMD:D_SOD-123, B.Cu at (148.7, 103.6)
- added D57: 1N4148W, Diode_SMD:D_SOD-123, B.Cu at (186.8, 103.6)
- added D58: 1N4148W, Diode_SMD:D_SOD-123, B.Cu at (224.9, 103.6)
- added D59: 1N4148W, Diode_SMD:D_SOD-123, B.Cu at (263.0, 103.6)
- added D6: 1N4148W, Diode_SMD:D_SOD-123, B.Cu at (258.3, 41.7)
- added D60: 1N4148W, Diode_SMD:D_SOD-123, B.Cu at (301.1, 103.6)
- added D61: 1N4148W, Diode_SMD:D_SOD-123, B.Cu at (405.9, 103.6)
- added D62: 1N4148W, Diode_SMD:D_SOD-123, B.Cu at (153.5, 122.6)
- added D63: 1N4148W, Diode_SMD:D_SOD-123, B.Cu at (191.6, 122.6)
- added D64: 1N4148W, Diode_SMD:D_SOD-123, B.Cu at (229.7, 122.6)
- added D65: 1N4148W, Diode_SMD:D_SOD-123, B.Cu at (267.8, 122.6)
- added D66: 1N4148W, Diode_SMD:D_SOD-123, B.Cu at (305.9, 122.6)
- added D67: 1N4148W, Diode_SMD:D_SOD-123, B.Cu at (344.0, 122.6)
- added D68: 1N4148W, Diode_SMD:D_SOD-123, B.Cu at (363.0, 122.6)
- added D69: 1N4148W, Diode_SMD:D_SOD-123, B.Cu at (358.3, 103.6)
- added D7: 1N4148W, Diode_SMD:D_SOD-123, B.Cu at (301.1, 41.7)
- added D70: 1N4148W, Diode_SMD:D_SOD-123, B.Cu at (124.9, 122.6)
- added D71: 1N4148W, Diode_SMD:D_SOD-123, B.Cu at (172.5, 122.6)
- added D72: 1N4148W, Diode_SMD:D_SOD-123, B.Cu at (210.6, 122.6)
- added D73: 1N4148W, Diode_SMD:D_SOD-123, B.Cu at (248.7, 122.6)
- added D74: 1N4148W, Diode_SMD:D_SOD-123, B.Cu at (286.8, 122.6)
- added D75: 1N4148W, Diode_SMD:D_SOD-123, B.Cu at (324.9, 122.6)
- added D76: 1N4148W, Diode_SMD:D_SOD-123, B.Cu at (405.9, 122.6)
- added D77: 1N4148W, Diode_SMD:D_SOD-123, B.Cu at (144.0, 141.7)
- added D78: 1N4148W, Diode_SMD:D_SOD-123, B.Cu at (182.1, 141.7)
- added D79: 1N4148W, Diode_SMD:D_SOD-123, B.Cu at (241.6, 141.7)
- added D8: 1N4148W, Diode_SMD:D_SOD-123, B.Cu at (339.2, 41.7)
- added D80: 1N4148W, Diode_SMD:D_SOD-123, B.Cu at (301.1, 141.7)
- added D81: 1N4148W, Diode_SMD:D_SOD-123, B.Cu at (344.0, 141.7)
- added D82: 1N4148W, Diode_SMD:D_SOD-123, B.Cu at (382.1, 141.7)
- added D84: 1N4148W, Diode_SMD:D_SOD-123, B.Cu at (382.1, 122.6)
- added D85: 1N4148W, Diode_SMD:D_SOD-123, B.Cu at (117.8, 141.7)
- added D86: 1N4148W, Diode_SMD:D_SOD-123, B.Cu at (163.0, 141.7)
- added D87: 1N4148W, Diode_SMD:D_SOD-123, B.Cu at (201.1, 141.7)
- added D88: 1N4148W, Diode_SMD:D_SOD-123, B.Cu at (282.1, 141.7)
- added D89: 1N4148W, Diode_SMD:D_SOD-123, B.Cu at (320.2, 141.7)
- added D9: 1N4148W, Diode_SMD:D_SOD-123, B.Cu at (382.1, 41.7)
- added D90: 1N4148W, Diode_SMD:D_SOD-123, B.Cu at (363.0, 141.7)
- added EN1: RotaryEncoder_Switch, BrownSugar_KBD:RotaryEncoder_EC11-Switch, F.Cu at (43.8, 85.8)
- added EN2: RotaryEncoder_Switch, BrownSugar_KBD:RotaryEncoder_EC11-Switch, F.Cu at (83.8, 85.8)
- added EN3: RotaryEncoder_Switch, BrownSugar_KBD:RotaryEncoder_EC11-Switch, F.Cu at (63.8, 122.8)
- added Q6: MMBT3906, Package_TO_SOT_SMD:SOT-23, B.Cu at (31.1, 70.5)
- added R12: 10k, Resistor_SMD:R_0603_1608Metric_Pad0.98x0.95mm_HandSolder, B.Cu at (51.4, 90.3)
- added R13: 10k, Resistor_SMD:R_0603_1608Metric_Pad0.98x0.95mm_HandSolder, B.Cu at (51.4, 81.4)
- added R14: 10k, Resistor_SMD:R_0603_1608Metric_Pad0.98x0.95mm_HandSolder, B.Cu at (76.2, 81.3)
- added R15: 10k, Resistor_SMD:R_0603_1608Metric_Pad0.98x0.95mm_HandSolder, B.Cu at (76.2, 90.3)
- added R16: 10k, Resistor_SMD:R_0603_1608Metric_Pad0.98x0.95mm_HandSolder, B.Cu at (57.4, 129.3)
- added R17: 10k, Resistor_SMD:R_0603_1608Metric_Pad0.98x0.95mm_HandSolder, B.Cu at (70.1, 129.3)
- added R18: 10k, Resistor_SMD:R_0603_1608Metric_Pad0.98x0.95mm_HandSolder, B.Cu at (49.0, 89.3)
- added R19: 10k, Resistor_SMD:R_0603_1608Metric_Pad0.98x0.95mm_HandSolder, B.Cu at (49.0, 82.6)
- added R20: 10k, Resistor_SMD:R_0603_1608Metric_Pad0.98x0.95mm_HandSolder, B.Cu at (78.6, 82.4)
- added R21: 10k, Resistor_SMD:R_0603_1608Metric_Pad0.98x0.95mm_HandSolder, B.Cu at (78.6, 89.3)
- added R22: 10k, Resistor_SMD:R_0603_1608Metric_Pad0.98x0.95mm_HandSolder, B.Cu at (59.2, 129.3)
- added R23: 10k, Resistor_SMD:R_0603_1608Metric_Pad0.98x0.95mm_HandSolder, B.Cu at (68.3, 129.3)
- added R24: 10k, Resistor_SMD:R_0603_1608Metric_Pad0.98x0.95mm_HandSolder, B.Cu at (38.9, 84.5)
- added R25: 10k, Resistor_SMD:R_0603_1608Metric_Pad0.98x0.95mm_HandSolder, B.Cu at (88.8, 87.2)
- added R26: 10k, Resistor_SMD:R_0603_1608Metric_Pad0.98x0.95mm_HandSolder, B.Cu at (65.3, 117.9)
- added REF**: MountingHole_3.2mm_M3_DIN965, MountingHole:MountingHole_3.2mm_M3_DIN965, F.Cu at (32.1, 56.1)
- added REF**: MountingHole_3.2mm_M3_DIN965, MountingHole:MountingHole_3.2mm_M3_DIN965, F.Cu at (32.1, 149.5)
- added S1: BOOT, SKRPACE010:SW_SKRPACE010, F.Cu at (63.2, 55.5)
- added S2: RST, SKRPACE010:SW_SKRPACE010, F.Cu at (54.0, 55.4)
- added SW10: SW_PUSH, BrownSugar_KBD:CherryMX_Hotswap_via_1U, F.Cu at (293.6, 42.2)
- added SW11: SW_PUSH, BrownSugar_KBD:CherryMX_Hotswap_via_1U, F.Cu at (312.7, 42.2)
- added SW12: SW_PUSH, BrownSugar_KBD:CherryMX_Hotswap_via_1U, F.Cu at (331.7, 42.2)
- added SW13: SW_PUSH, BrownSugar_KBD:CherryMX_Hotswap_via_1U, F.Cu at (350.8, 42.2)
- added SW14: SW_PUSH, BrownSugar_KBD:CherryMX_Hotswap_via_1U, F.Cu at (374.6, 42.2)
- added SW15: SW_PUSH, BrownSugar_KBD:CherryMX_Hotswap_via_1U, F.Cu at (398.4, 42.2)
- added SW16: SW_PUSH, BrownSugar_KBD:CherryMX_Hotswap_via_1U, F.Cu at (107.9, 66.0)
- added SW17: SW_PUSH, BrownSugar_KBD:CherryMX_Hotswap_via_1U, F.Cu at (126.9, 66.0)
- added SW18: SW_PUSH, BrownSugar_KBD:CherryMX_Hotswap_via_1U, F.Cu at (146.0, 66.0)
- added SW19: SW_PUSH, BrownSugar_KBD:CherryMX_Hotswap_via_1U, F.Cu at (165.0, 66.0)
- added SW20: SW_PUSH, BrownSugar_KBD:CherryMX_Hotswap_via_1U, F.Cu at (184.1, 66.0)
- added SW21: SW_PUSH, BrownSugar_KBD:CherryMX_Hotswap_via_1U, F.Cu at (203.1, 66.0)
- added SW22: SW_PUSH, BrownSugar_KBD:CherryMX_Hotswap_via_1U, F.Cu at (222.2, 66.0)
- added SW23: SW_PUSH, BrownSugar_KBD:CherryMX_Hotswap_via_1U, F.Cu at (241.2, 66.0)
- added SW24: SW_PUSH, BrownSugar_KBD:CherryMX_Hotswap_via_1U, F.Cu at (260.3, 66.0)
- added SW25: SW_PUSH, BrownSugar_KBD:CherryMX_Hotswap_via_1U, F.Cu at (279.3, 66.0)
- added SW26: SW_PUSH, BrownSugar_KBD:CherryMX_Hotswap_via_1U, F.Cu at (298.4, 66.0)
- added SW27: SW_PUSH, BrownSugar_KBD:CherryMX_Hotswap_via_1U, F.Cu at (317.4, 66.0)
- added SW28: SW_PUSH, BrownSugar_KBD:CherryMX_Hotswap_via_1U, F.Cu at (336.5, 66.0)
- added SW29: SW_PUSH, BrownSugar_KBD:CherryMX_Hotswap_via_1U, F.Cu at (355.5, 66.0)
- added SW3: SW_PUSH, BrownSugar_KBD:CherryMX_Hotswap_via_1U, F.Cu at (150.8, 42.2)
- added SW30: SW_PUSH, BrownSugar_KBD:CherryMX_Hotswap_via_1U, F.Cu at (374.6, 66.0)
- added SW31: SW_PUSH, BrownSugar_KBD:CherryMX_Hotswap_via_1U, F.Cu at (398.4, 66.0)
- added SW32: SW_PUSH, BrownSugar_KBD:CherryMX_Hotswap_via_1U, F.Cu at (112.7, 85.0)
- added SW33: SW_PUSH, BrownSugar_KBD:CherryMX_Hotswap_via_1U, F.Cu at (136.5, 85.0)
- added SW34: SW_PUSH, BrownSugar_KBD:CherryMX_Hotswap_via_1U, F.Cu at (155.5, 85.0)
- added SW35: SW_PUSH, BrownSugar_KBD:CherryMX_Hotswap_via_1U, F.Cu at (174.6, 85.0)
- added SW36: SW_PUSH, BrownSugar_KBD:CherryMX_Hotswap_via_1U, F.Cu at (193.6, 85.0)
- added SW37: SW_PUSH, BrownSugar_KBD:CherryMX_Hotswap_via_1U, F.Cu at (212.7, 85.0)
- added SW38: SW_PUSH, BrownSugar_KBD:CherryMX_Hotswap_via_1U, F.Cu at (231.7, 85.0)
- added SW39: SW_PUSH, BrownSugar_KBD:CherryMX_Hotswap_via_1U, F.Cu at (250.8, 85.0)
- added SW4: SW_PUSH, BrownSugar_KBD:CherryMX_Hotswap_via_1U, F.Cu at (169.8, 42.2)
- added SW40: SW_PUSH, BrownSugar_KBD:CherryMX_Hotswap_via_1U, F.Cu at (269.8, 85.0)
- added SW41: SW_PUSH, BrownSugar_KBD:CherryMX_Hotswap_via_1U, F.Cu at (288.9, 85.0)
- added SW42: SW_PUSH, BrownSugar_KBD:CherryMX_Hotswap_via_1U, F.Cu at (307.9, 85.0)
- added SW43: SW_PUSH, BrownSugar_KBD:CherryMX_Hotswap_via_1U, F.Cu at (327.0, 85.0)
- added SW44: SW_PUSH, BrownSugar_KBD:CherryMX_Hotswap_via_1U, F.Cu at (346.0, 85.0)
- added SW45: SW_PUSH, BrownSugar_KBD:CherryMX_Hotswap_via_1U, F.Cu at (372.2, 94.5)
- added SW46: SW_PUSH, BrownSugar_KBD:CherryMX_Hotswap_via_1U, F.Cu at (398.4, 85.0)
- added SW47: SW_PUSH, BrownSugar_KBD:CherryMX_Hotswap_via_1U, F.Cu at (115.0, 104.1)
- added SW48: SW_PUSH, BrownSugar_KBD:CherryMX_Hotswap_via_1U, F.Cu at (141.2, 104.1)
- added SW49: SW_PUSH, BrownSugar_KBD:CherryMX_Hotswap_via_1U, F.Cu at (160.3, 104.1)
- added SW5: SW_PUSH, BrownSugar_KBD:CherryMX_Hotswap_via_1U, F.Cu at (188.9, 42.2)
- added SW50: SW_PUSH, BrownSugar_KBD:CherryMX_Hotswap_via_1U, F.Cu at (179.3, 104.1)
- added SW51: SW_PUSH, BrownSugar_KBD:CherryMX_Hotswap_via_1U, F.Cu at (198.4, 104.1)
- added SW52: SW_PUSH, BrownSugar_KBD:CherryMX_Hotswap_via_1U, F.Cu at (217.4, 104.1)
- added SW53: SW_PUSH, BrownSugar_KBD:CherryMX_Hotswap_via_1U, F.Cu at (236.5, 104.1)
- added SW54: SW_PUSH, BrownSugar_KBD:CherryMX_Hotswap_via_1U, F.Cu at (255.5, 104.1)
- added SW55: SW_PUSH, BrownSugar_KBD:CherryMX_Hotswap_via_1U, F.Cu at (274.6, 104.1)
- added SW56: SW_PUSH, BrownSugar_KBD:CherryMX_Hotswap_via_1U, F.Cu at (293.6, 104.1)
- added SW57: SW_PUSH, BrownSugar_KBD:CherryMX_Hotswap_via_1U, F.Cu at (312.7, 104.1)
- added SW58: SW_PUSH, BrownSugar_KBD:CherryMX_Hotswap_via_1U, F.Cu at (331.7, 104.1)
- added SW59: SW_PUSH, BrownSugar_KBD:CherryMX_Hotswap_via_1U, F.Cu at (350.8, 104.1)
- added SW6: SW_PUSH, BrownSugar_KBD:CherryMX_Hotswap_via_1U, F.Cu at (212.7, 42.2)
- added SW60: SW_PUSH, BrownSugar_KBD:CherryMX_Hotswap_via_1U, F.Cu at (398.4, 104.1)
- added SW61: SW_PUSH, BrownSugar_KBD:CherryMX_Hotswap_via_1U, F.Cu at (117.4, 123.1)
- added SW62: SW_PUSH, BrownSugar_KBD:CherryMX_Hotswap_via_1U, F.Cu at (146.0, 123.1)
- added SW63: SW_PUSH, BrownSugar_KBD:CherryMX_Hotswap_via_1U, F.Cu at (165.0, 123.1)
- added SW64: SW_PUSH, BrownSugar_KBD:CherryMX_Hotswap_via_1U, F.Cu at (184.1, 123.1)
- added SW65: SW_PUSH, BrownSugar_KBD:CherryMX_Hotswap_via_1U, F.Cu at (203.1, 123.1)
- added SW66: SW_PUSH, BrownSugar_KBD:CherryMX_Hotswap_via_1U, F.Cu at (222.2, 123.1)
- added SW67: SW_PUSH, BrownSugar_KBD:CherryMX_Hotswap_via_1U, F.Cu at (241.2, 123.1)
- added SW68: SW_PUSH, BrownSugar_KBD:CherryMX_Hotswap_via_1U, F.Cu at (260.3, 123.1)
- added SW69: SW_PUSH, BrownSugar_KBD:CherryMX_Hotswap_via_1U, F.Cu at (279.3, 123.1)
- added SW7: SW_PUSH, BrownSugar_KBD:CherryMX_Hotswap_via_1U, F.Cu at (231.7, 42.2)
- added SW70: SW_PUSH, BrownSugar_KBD:CherryMX_Hotswap_via_1U, F.Cu at (298.4, 123.1)
- added SW71: SW_PUSH, BrownSugar_KBD:CherryMX_Hotswap_via_1U, F.Cu at (317.4, 123.1)
- added SW72: SW_PUSH, BrownSugar_KBD:CherryMX_Hotswap_via_1U, F.Cu at (336.5, 123.1)
- added SW73: SW_PUSH, BrownSugar_KBD:CherryMX_Hotswap_via_1U, F.Cu at (355.5, 123.1)
- added SW74: SW_PUSH, BrownSugar_KBD:CherryMX_Hotswap_via_1U, F.Cu at (374.6, 123.1)
- added SW75: SW_PUSH, BrownSugar_KBD:CherryMX_Hotswap_via_1U, F.Cu at (398.4, 123.1)
- added SW76: SW_PUSH, BrownSugar_KBD:CherryMX_Hotswap_via_1U, F.Cu at (110.3, 142.2)
- added SW77: SW_PUSH, BrownSugar_KBD:CherryMX_Hotswap_via_1U, F.Cu at (136.5, 142.2)
- added SW78: SW_PUSH, BrownSugar_KBD:CherryMX_Hotswap_via_1U, F.Cu at (155.5, 142.2)
- added SW79: SW_PUSH, BrownSugar_KBD:CherryMX_Hotswap_via_1U, F.Cu at (174.6, 142.2)
- added SW8: SW_PUSH, BrownSugar_KBD:CherryMX_Hotswap_via_1U, F.Cu at (250.8, 42.2)
- added SW80: SW_PUSH, BrownSugar_KBD:CherryMX_Hotswap_via_1U, F.Cu at (193.6, 142.2)
- added SW81: SW_PUSH, BrownSugar_KBD:CherryMX_Hotswap_via_1U, F.Cu at (234.1, 142.2)
- added SW82: SW_PUSH, BrownSugar_KBD:CherryMX_Hotswap_via_1U, F.Cu at (274.6, 142.2)
- added SW83: SW_PUSH, BrownSugar_KBD:CherryMX_Hotswap_via_1U, F.Cu at (293.6, 142.2)
- added SW84: SW_PUSH, BrownSugar_KBD:CherryMX_Hotswap_via_1U, F.Cu at (312.7, 142.2)
- added SW85: SW_PUSH, BrownSugar_KBD:CherryMX_Hotswap_via_1U, F.Cu at (336.5, 142.2)
- added SW86: SW_PUSH, BrownSugar_KBD:CherryMX_Hotswap_via_1U, F.Cu at (355.5, 142.2)
- added SW87: SW_PUSH, BrownSugar_KBD:CherryMX_Hotswap_via_1U, F.Cu at (374.6, 142.2)
- added SW9: SW_PUSH, BrownSugar_KBD:CherryMX_Hotswap_via_1U, F.Cu at (269.8, 42.2)
- added U4: ESP32-S3-WROOM-1, RF_Module:ESP32-S3-WROOM-1, B.Cu at (58.9, 59.1)
- C1: value 47uF -> 0.1uF; footprint Capacitor_SMD:CP_Elec_6.3x4.5 -> Capacitor_SMD:C_0603_1608Metric_Pad1.08x0.95mm_HandSolder; moved to B.Cu
- C2: value 0.33uF -> 0.1uF; moved to B.Cu
- C3: value 0.1uF -> 10uF; moved to B.Cu
- C5, C7: value 0.1uF -> 22uF; moved to B.Cu
- C8: value 22uF -> 0.1uF; moved to B.Cu
- J1: footprint Connector_JST:JST_XH_S2B-XH-A_1x02_P2.50mm_Horizontal -> Connector_PinHeader_2.54mm:PinHeader_1x02_P2.54mm_Vertical; moved to B.Cu
- J2, Q3, R3, R5, R6, R7, R8: moved to B.Cu
- Q1, Q2: value MMBT3906 -> BSS138; moved to B.Cu
- Q4, Q5: value BSS138 -> MMBT3906; moved to B.Cu
- R1: value 10k -> 5k; moved to B.Cu
- R10, R9: value 5k -> 10k; moved to B.Cu
- R2: value 10k -> 5.1k; moved to B.Cu
- R4: value 5.1k -> 5k; moved to B.Cu
- SW1: value BOOT -> SW_PUSH; footprint SKRPACE010:SW_SKRPACE010 -> BrownSugar_KBD:CherryMX_Hotswap_via_1U
- SW2: value RST -> SW_PUSH; footprint SKRPACE010:SW_SKRPACE010 -> BrownSugar_KBD:CherryMX_Hotswap_via_1U
- U1: value FDS4935A -> CH340K; footprint footprints:SO-8_ONS-L -> Package_SO:SSOP-10-1EP_3.9x4.9mm_P1mm_EP2.1x3.3mm; moved to B.Cu
- U2: value ESP32-S3-WROOM-1 -> FDS4935A; footprint RF_Module:ESP32-S3-WROOM-1 -> footprints:SO-8_ONS-L; moved to B.Cu
- U3: value CH340K -> AZ1117CH-3.3TRG1; footprint Package_SO:SSOP-10-1EP_3.9x4.9mm_P1mm_EP2.1x3.3mm -> AZ1117CH_3_3TRG1:SOT-223_DIO-M; moved to B.Cu
- moved SW2 85.8 mm to (131.7, 42.2)
- moved Q1 71.4 mm to (47.3, 73.2), turned to -90 degrees
- moved Q2 67.1 mm to (43.9, 73.2), turned to -90 degrees
- moved SW1 61.5 mm to (107.9, 42.2)
- moved C7 59.2 mm to (72.4, 55.1), turned to 90 degrees
- moved C8 56.4 mm to (69.5, 55.0), turned to 90 degrees
- moved Q3 55.7 mm to (39.8, 65.7), turned to 90 degrees
- moved Q4 54.4 mm to (31.1, 66.4), turned to -90 degrees
- moved Q5 50.6 mm to (39.8, 69.7), turned to 90 degrees
- moved C4 46.7 mm to (59.4, 55.4), turned to 90 degrees
- moved R11 45.2 mm to (66.9, 55.5), turned to 90 degrees
- moved C6 44.7 mm to (57.8, 55.4), turned to 90 degrees
- moved U2 41.6 mm to (35.5, 67.8), turned to 90 degrees
- moved C2 38.4 mm to (42.7, 67.6), turned to 90 degrees
- moved C3 35.1 mm to (35.7, 72.5)
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Connections:
- C1 pad 1: +3.3V -> VDD
- C2 pad 1: VDD -> Net-(U1-V3)
- C4 pad 1: Net-(U3-V3) -> /ESP32-S3/en
- C5 pad 1: /ESP32-S3/en -> +3.3V
- Q1 pad 1: Net-(Q1-B) -> Net-(Q1-G)
- Q1 pad 2: Net-(J1-Pin_2) -> /ESP32-S3/RTS
- Q1 pad 3: Net-(Q1-B) -> /ESP32-S3/en
- Q2 pad 1: Net-(Q1-B) -> Net-(Q2-G)
- Q2 pad 2: VDD -> /ESP32-S3/DTR
- Q2 pad 3: Net-(Q2-C) -> /ESP32-S3/IO0
- Q4 pad 1: Net-(Q4-G) -> Net-(Q4-B)
- Q4 pad 2: /ESP32-S3/DTR -> Net-(J1-Pin_2)
- Q4 pad 3: /ESP32-S3/IO0 -> Net-(Q4-B)
- Q5 pad 1: Net-(Q5-G) -> Net-(Q3-B)
- Q5 pad 2: /ESP32-S3/RTS -> VDD
- Q5 pad 3: /ESP32-S3/en -> Net-(Q5-C)
- R1 pad 1: Net-(Q3-B) -> Net-(D1-A)
- R1 pad 2: GND -> Net-(J1-Pin_2)
- R10 pad 1: Net-(D2-A) -> Net-(Q6-C)
- R10 pad 2: Net-(Q3-E) -> GND
- R2 pad 1: Net-(Q7-C) -> Net-(J2-CC1)
- R3 pad 1: Net-(J2-CC1) -> Net-(J2-CC2)
- R4 pad 1: Net-(J2-CC2) -> Net-(D2-A)
- R4 pad 2: GND -> Net-(Q3-E)
- R5 pad 1: GND -> /ESP32-S3/DTR
- R5 pad 2: Net-(Q1-B) -> Net-(Q1-G)
- R6 pad 1: GND -> /ESP32-S3/RTS
- R6 pad 2: Net-(Q2-C) -> Net-(Q2-G)
- R7 pad 1: /ESP32-S3/DTR -> GND
- R7 pad 2: Net-(Q5-G) -> Net-(Q3-B)
- R8 pad 1: /ESP32-S3/RTS -> Net-(Q4-B)
- R8 pad 2: Net-(Q4-G) -> GND
- R9 pad 1: Net-(D1-A) -> GND
- R9 pad 2: Net-(J1-Pin_2) -> Net-(Q5-C)
- SW1 pad 1: GND -> /ESP32-S3/IO4
- SW1 pad 2: /ESP32-S3/en -> Net-(D10-K)
- SW2 pad 1: GND -> /ESP32-S3/IO4
- SW2 pad 2: /ESP32-S3/IO0 -> Net-(D3-A)
- U1 pad 1: VDD -> /ESP32-S3/D+
- U1 pad 2: Net-(Q2-C) -> /ESP32-S3/D-
- U1 pad 3: VDD -> GND
- U1 pad 4: Net-(Q7-C) -> /ESP32-S3/DTR
- U1 pad 5: Net-(Q3-E) -> unconnected-(U1-~{CTS}-Pad5)
- U1 pad 6: Net-(Q3-E) -> /ESP32-S3/RTS
- U1 pad 7: Net-(J1-Pin_2) -> VDD
- U1 pad 8: Net-(J1-Pin_2) -> /ESP32-S3/RX
- U2 pad 1: GND -> VDD
- U2 pad 2: +3.3V -> Net-(Q5-C)
- U2 pad 3: /ESP32-S3/en -> VDD
- U2 pad 4: unconnected-(U2-IO4-Pad4) -> Net-(Q6-C)
- U2 pad 5: unconnected-(U2-IO5-Pad5) -> Net-(J1-Pin_2)
- U2 pad 6: unconnected-(U2-IO6-Pad6) -> Net-(J1-Pin_2)
- U2 pad 7: unconnected-(U2-IO7-Pad7) -> Net-(Q3-E)
- U2 pad 8: unconnected-(U2-IO15-Pad8) -> Net-(Q3-E)
- U3 pad 1: /ESP32-S3/D+ -> GND
- U3 pad 2: /ESP32-S3/D- -> +3.3V
- U3 pad 3: GND -> VDD
- U3 pad 4: /ESP32-S3/DTR -> unconnected-(U3-EPAD-Pad4)
Routing:
- net +3.3V: track 0.00 -> 194.0 mm, vias 0 -> 6
- net /ESP32-S3/enc3_B_IO1: track 0.00 -> 82.8 mm, vias 0 -> 4
- net /ESP32-S3/enc3_A_IO2: track 0.00 -> 77.9 mm, vias 0 -> 2
- net /ESP32-S3/enc3_SW_IO47: track 0.00 -> 51.3 mm, vias 0 -> 2
- net /ESP32-S3/enc2_B_IO40: track 0.00 -> 50.7 mm, vias 0 -> 2
- net /ESP32-S3/enc2_SW_IO48: track 0.00 -> 48.7 mm
- net /ESP32-S3/en: track 0.00 -> 43.9 mm, vias 0 -> 4
- net /ESP32-S3/enc2_A_IO39: track 0.00 -> 41.2 mm, vias 0 -> 2
- net /ESP32-S3/IO0: track 0.00 -> 32.2 mm, vias 0 -> 3
- net VDD: track 0.00 -> 31.4 mm, vias 0 -> 2
- net /ESP32-S3/enc1_A_IO41: track 0.00 -> 30.8 mm, vias 0 -> 2
- net /ESP32-S3/enc1_SW_IO38: track 0.00 -> 28.3 mm, vias 0 -> 2
- net /ESP32-S3/enc1_B_IO42: track 0.00 -> 24.3 mm, vias 0 -> 2
- net GND: track 0.00 -> 23.6 mm, vias 0 -> 94
- net Net-(Q3-E): track 0.00 -> 20.2 mm, vias 0 -> 4
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Other:
- board outline added: 380.2 x 121.1 mm
