File: Davinci-Keyboard/Davinci-Keyboard.kicad_sch (KiCad schematic)
At the start: 0 parts

Commit message: 20$越え
Connections:
- no-connect marks 0 -> 2
Other:
- sheet ESP32-S3 ports: added IO17, IO18, enc1_SW_IO38, enc2_SW_IO48, enc3_A_IO2, enc3_B_IO1, enc3_SW_IO47; removed IO1, IO2, IO47, IO48, enc3_A_IO17, enc3_B_IO18
- sheet Key Switches ports: added IO10, IO11, IO12, IO13, IO15, IO16, IO17, IO18, IO4, IO5, IO6, IO7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; removed none
- sheet RotaryEncoder ports: added enc1_SW, enc2_SW, enc3_SW; removed none
