File: Davinci-Keyboard/esp32_s3.kicad_sch (KiCad schematic)
At the start: 35 parts, among them J1 Conn_01x02, J2 USB_C_Receptacle_USB2.0_16P, Q1 MMBT3906, Q2 MMBT3906, Q3 MMBT3906, Q4 BSS138, Q5 BSS138, Q7 MMBT3906, U1 FDS4935A, U2 ESP32-S3-WROOM-1, U3 CH340K

Commit message: 20$越え
Parts:
- removed C1: 47uF, Capacitor_SMD:CP_Elec_6.3x4.5, symbol Device:C_Polarized_Small
- removed LDO1: ~, Package_TO_SOT_THT:TO-220-4_Horizontal_TabDown, symbol MyLibrary:PQ3RD23
- added C5: 22uF, Capacitor_SMD:C_0603_1608Metric_Pad1.08x0.95mm_HandSolder, symbol Device:C_Small
- added U3: AZ1117CH-3.3TRG1, AZ1117CH_3_3TRG1:SOT-223_DIO-M, symbol 2024-12-31_11-23-54:AZ1117CH-3.3TRG1
- C3: renamed from C2; value 0.33uF -> 10uF
- J1: footprint Connector_JST:JST_XH_S2B-XH-A_1x02_P2.50mm_Horizontal -> Connector_PinHeader_2.54mm:PinHeader_1x02_P2.54mm_Vertical
- renumbered C3 to C1, C4 to C2, C5 to C4, C8 to C7, C7 to C8, Q5 to Q1, Q4 to Q2, Q1 to Q3, Q3 to Q4, Q2 to Q5, Q7 to Q6, R9 to R1, R2 to R10, R3 to R2, R4 to R3, R10 to R4, R7 to R5, R8 to R6, R5 to R7, R1 to R8, R6 to R9, U3 to U1, U1 to U2, U2 to U4
Connections:
- net +3.3V: now also C5.1, U3.2 (OUTPUT)
- net GND: now also S1.2, S2.2, C5.2, U3.1 (ADJ/GND); no longer S1.3, S2.3
- net IO0: now also S2.3; no longer S2.2
- net VDD: now also U3.3 (INPUT)
- net en: now also S1.3; no longer S1.2
- net enc1_SW_IO38: now reaches U4.31 (IO38)
- net at Q3.2 (E), U2.7 (D2), U2.8 (D2): now also J2.A4 (VBUS), J2.A9 (VBUS), J2.B4 (VBUS), J2.B9 (VBUS), R4.2; no longer J1.2 (Pin_2), R1.2
- net IO1 renamed enc3_B_IO1
- net IO2 renamed enc3_A_IO2
- net IO47 renamed enc3_SW_IO47
- net IO48 renamed enc2_SW_IO48
- net enc3_A_IO17 renamed IO17
- net enc3_B_IO18 renamed IO18
- new net: J1.2 (Pin_2), Q4.2 (E), R1.2, U2.5 (D1), U2.6 (D1)
- no-connect marks 13 -> 12
Other:
- note removed: "can use"
- moved on the sheet: C4, C6
