File: Davinci-Keyboard/sw.kicad_sch (KiCad schematic)
At the start: 0 parts

Commit message: 20$越え
Parts:
- added D10, D11, D12, D13, D14, D15, D16, D17, D18, D19, D20, D21, D22, D23, D24, D25, D26, D27, D28, D29, D3, D30, D31, D32, D33, D34, D35, D36, D37, D38, D39, D4, D40, D41, D42, D43, D44, D45, D46, D47, D48, D49, D5, D50, D51, D52, D53, D54, D55, D56, D57, D58, D59, D6, D60, D61, D62, D63, D64, D65, D66, D67, D68, D69, D7, D70, D71, D72, D73, D74, D75, D76, D77, D78, D79, D8, D80, D81, D82, D84, D85, D86, D87, D88, D89, D9, D90: 1N4148W, Diode_SMD:D_SOD-123, symbol Diode:1N4148W
- added SW1, SW10, SW11, SW12, SW13, SW14, SW15, SW16, SW17, SW18, SW19, SW2, SW20, SW21, SW22, SW23, SW24, SW25, SW26, SW27, SW28, SW29, SW3, SW30, SW31, SW32, SW33, SW34, SW35, SW36, SW37, SW38, SW39, SW4, SW40, SW41, SW42, SW43, SW44, SW45, SW46, SW47, SW48, SW49, SW5, SW50, SW51, SW52, SW53, SW54, SW55, SW56, SW57, SW58, SW59, SW6, SW60, SW61, SW62, SW63, SW64, SW65, SW66, SW67, SW68, SW69, SW7, SW70, SW71, SW72, SW73, SW74, SW75, SW76, SW77, SW78, SW79, SW8, SW80, SW81, SW82, SW83, SW84, SW85, SW86, SW87, SW9: SW_PUSH, CherryMX_Hotswap_via_1U, symbol BrownSugar_KBD:SW_PUSH
Connections:
- new net: D34.2 (A), SW36.2
- new net: D19.2 (A), SW20.2
- new net: D82.2 (A), SW87.2
- new net: D72.1 (K), SW65.2
- new net: D21.2 (A), SW24.2
- new net: D16.1 (K), SW13.2
- new net: D79.2 (A), SW81.2
- new net: D22.2 (A), SW26.2
- new net: D56.1 (K), SW48.2
- new net: D3.2 (A), SW2.2
- new net: D43.1 (K), SW37.2
- new net: D9.2 (A), SW14.2
- new net: D89.1 (K), SW84.2
- new net: D45.1 (K), SW41.2
- new net: D7.2 (A), SW10.2
- new net: D54.1 (K), SW44.2
- new net: D64.2 (A), SW66.2
- new net: D11.1 (K), SW3.2
- new net: D47.2 (A), SW47.2
- new net: D65.2 (A), SW68.2
- new net: D42.1 (K), SW35.2
- new net: D35.2 (A), SW38.2
- new net: D85.1 (K), SW76.2
- new net: D8.2 (A), SW12.2
- new net: D81.2 (A), SW85.2
- new net: D75.1 (K), SW71.2
- new net: D24.1 (K), SW15.2
- new net: D26.1 (K), SW19.2
- new net: D52.2 (A), SW57.2
- new net: D23.2 (A), SW28.2
- new net: D10.1 (K), SW1.2
- new net: D5.2 (A), SW6.2
- new net: D55.1 (K), SW46.2
- new net: D46.2 (A), SW45.2
- new net: D44.1 (K), SW39.2
- new net: D66.2 (A), SW70.2
- new net: D63.2 (A), SW64.2
- new net: D51.2 (A), SW55.2
- new net: D84.1 (K), SW74.2
- new net: D20.2 (A), SW22.2
- new net: D78.2 (A), SW79.2
- new net: D53.2 (A), SW58.2
- new net: D73.1 (K), SW67.2
- new net: D58.1 (K), SW52.2
- new net: D15.1 (K), SW11.2
- new net: D4.2 (A), SW4.2
- new net: D12.1 (K), SW5.2
- new net: D48.2 (A), SW49.2
- new net: D38.2 (A), SW43.2
- new net: D62.2 (A), SW62.2
- new net: D50.2 (A), SW53.2
- new net: D27.1 (K), SW21.2
- new net: D60.1 (K), SW56.2
- new net: D37.2 (A), SW42.2
- new net: D40.1 (K), SW31.2
- new net: D30.1 (K), SW27.2
- new net: D88.1 (K), SW82.2
- new net: D28.1 (K), SW23.2
- new net: D57.1 (K), SW50.2
- new net: D6.2 (A), SW8.2
- new net: D76.2 (A), SW75.2
- new net: D25.1 (K), SW17.2
- new net: D87.1 (K), SW80.2
- new net: D13.1 (K), SW7.2
- new net: D32.2 (A), SW32.2
- new net: D39.1 (K), SW29.2
- new net: D59.1 (K), SW54.2
- new net: D80.2 (A), SW83.2
- new net: D90.1 (K), SW86.2
- new net: D29.1 (K), SW25.2
- new net: D49.2 (A), SW51.2
- new net: D31.2 (A), SW30.2
- new net: D74.1 (K), SW69.2
- new net: D68.2 (A), SW73.2
- new net: D77.2 (A), SW77.2
- new net: D18.2 (A), SW18.2
- new net: D33.2 (A), SW34.2
- new net: D41.1 (K), SW33.2
- new net: D71.1 (K), SW63.2
- new net: D70.1 (K), SW61.2
- new net: D86.1 (K), SW78.2
- new net: D61.2 (A), SW60.2
- new net: D14.1 (K), SW9.2
- new net: D17.2 (A), SW16.2
- new net: D67.2 (A), SW72.2
- new net: D36.2 (A), SW40.2
- new net: D69.1 (K), SW59.2
- new net IO10: D14.2 (A), D21.1 (K), D28.2 (A), D35.1 (K), D43.2 (A), D50.1 (K), D58.2 (A), D65.1 (K), D7.1 (K), D73.2 (A), D80.1 (K), D88.2 (A)
- new net IO11: D15.2 (A), D22.1 (K), D29.2 (A), D36.1 (K), D44.2 (A), D51.1 (K), D59.2 (A), D66.1 (K), D74.2 (A), D8.1 (K), D81.1 (K), D89.2 (A)
- new net IO12: D16.2 (A), D23.1 (K), D30.2 (A), D37.1 (K), D45.2 (A), D52.1 (K), D60.2 (A), D67.1 (K), D75.2 (A), D82.1 (K), D9.1 (K), D90.2 (A)
- new net IO13: D38.1 (K), D53.1 (K), D68.1 (K)
- new net IO15: SW59.1, SW60.1, SW61.1, SW62.1, SW63.1, SW64.1, SW65.1, SW66.1, SW67.1, SW68.1, SW69.1, SW70.1, SW71.1, SW72.1, SW73.1
- new net IO16: SW74.1, SW75.1, SW76.1, SW77.1, SW78.1, SW79.1, SW80.1, SW81.1, SW82.1, SW83.1, SW84.1, SW85.1, SW86.1, SW87.1
- new net IO17: D10.2 (A), D17.1 (K), D24.2 (A), D3.1 (K), D31.1 (K), D39.2 (A), D46.1 (K), D54.2 (A), D61.1 (K), D69.2 (A), D76.1 (K), D84.2 (A)
- new net IO18: D11.2 (A), D18.1 (K), D25.2 (A), D32.1 (K), D4.1 (K), D40.2 (A), D47.1 (K), D55.2 (A), D62.1 (K), D70.2 (A), D77.1 (K), D85.2 (A)
- new net IO4: SW1.1, SW10.1, SW11.1, SW12.1, SW13.1, SW14.1, SW2.1, SW3.1, SW4.1, SW5.1, SW6.1, SW7.1, SW8.1, SW9.1
- new net IO5: SW15.1, SW16.1, SW17.1, SW18.1, SW19.1, SW20.1, SW21.1, SW22.1, SW23.1, SW24.1, SW25.1, SW26.1, SW27.1, SW28.1
- new net IO6: SW29.1, SW30.1, SW31.1, SW32.1, SW33.1, SW34.1, SW35.1, SW36.1, SW37.1, SW38.1, SW39.1, SW40.1, SW41.1, SW42.1, SW43.1
- new net IO7: SW44.1, SW45.1, SW46.1, SW47.1, SW48.1, SW49.1, SW50.1, SW51.1, SW52.1, SW53.1, SW54.1, SW55.1, SW56.1, SW57.1, SW58.1
- new net IO8: D12.2 (A), D19.1 (K), D26.2 (A), D33.1 (K), D41.2 (A), D48.1 (K), D5.1 (K), D56.2 (A), D63.1 (K), D71.2 (A), D78.1 (K), D86.2 (A)
- new net IO9: D13.2 (A), D20.1 (K), D27.2 (A), D34.1 (K), D42.2 (A), D49.1 (K), D57.2 (A), D6.1 (K), D64.1 (K), D72.2 (A), D79.1 (K), D87.2 (A)
